File: fc-dumper-base-hat-2/fc-dumper-base-hat-2.kicad_sch (KiCad schematic)
At the start: 7 parts, among them J1 GPIO, J2 Conn_01x10_Male, J3 Conn_01x12_Male, U1 FXMA108, U2 74HC244

Commit message: update design, and document
Parts:
- removed JP1, JP2: SolderJumper_3_Open, Jumper:SolderJumper-3_P1.3mm_Open_RoundedPad1.0x1.5mm_NumberLabels, symbol Jumper:SolderJumper_3_Open
- added J4: Conn_01x04_Male, Connector_PinHeader_2.54mm:PinHeader_1x04_P2.54mm_Vertical, symbol Connector:Conn_01x04_Male
Connections:
- net GPIO2(SDA1) is gone; now on net EIO_0: J1.3 (Pin_3)
- net GPIO3(SCL1) is gone; now on net EIO_1: J1.5 (Pin_5)
- net EIO_0: now also J3.11 (Pin_11); no longer J3.8 (Pin_8)
- net EIO_1: now also J4.1 (Pin_1); no longer J3.9 (Pin_9)
- net EIO_2: now also J4.2 (Pin_2); no longer J3.11 (Pin_11)
- net EXT0 renamed PPUWR
- net PPUWR: now also J3.8 (Pin_8)
- net EXT1 renamed EXT
- net EXT: now also J3.9 (Pin_9)
- net GPIO[16] renamed EIO_3
- net EIO_3: now also J4.3 (Pin_3)
- net GPIO[26] renamed EIO_4
- net EIO_4: now also J4.4 (Pin_4)
- net RST renamed PPURD
- no-connect marks 7 -> 5
Other:
- moved on the sheet: J2, J3
