File: fc-dumper-base-hat-2/fc-dumper-base-hat-2.kicad_pcb (KiCad board)
At the start: 2 copper layers, 65 x 56 mm, 11 parts, among them J1 GPIO, J2 Conn_01x10_Male, J3 Conn_01x12_Male, U1 FXMA108, U2 74HC244

Commit message: update design, and document
Parts:
- removed JP1, JP2: SolderJumper_3_Open, Jumper:SolderJumper-3_P1.3mm_Open_RoundedPad1.0x1.5mm_NumberLabels
- added J4: Conn_01x04_Male, Connector_PinHeader_2.54mm:PinHeader_1x04_P2.54mm_Vertical, F.Cu at (150.8, 86.0)
- moved J3 34.2 mm to (154.6, 65.7)
- moved U1 29.2 mm to (118.4, 68.3)
- moved J2 17.9 mm to (108.9, 68.2)
- moved U2 8.77 mm to (134.3, 68.3)
Connections:
- net RST renamed PPURD
- J1 pad 3: /GPIO2(SDA1) -> EIO_0
- J1 pad 36: /GPIO[16] -> EIO_3
- J1 pad 37: /GPIO[26] -> EIO_4
- J1 pad 5: /GPIO3(SCL1) -> EIO_1
- J3 pad 11: EIO_2 -> EIO_0
- J3 pad 8: EIO_0 -> PPUWR
- J3 pad 9: EIO_1 -> EXT
- U2 pad 7: EXT0 -> PPUWR
- U2 pad 9: EXT1 -> EXT
Routing:
- net GND: track 0.00 -> 208.8 mm
- net PWM1: track 0.00 -> 113.9 mm
- net PWR3: track 0.00 -> 106.7 mm
- net EIO_0: track 0.00 -> 98.1 mm
- net EIO_1: track 0.00 -> 80.7 mm, vias 0 -> 1
- net PWM0: track 0.00 -> 78.5 mm
- net /GPIO25(GEN6): track 0.00 -> 74.0 mm, vias 0 -> 1
- net /GPIO7(SPI1_CE_N): track 0.00 -> 71.9 mm
- net /GPIO5: track 0.00 -> 70.0 mm
- net PWR: track 0.00 -> 64.5 mm, vias 0 -> 1
- net /GPIO24(GEN5): track 0.00 -> 58.8 mm
- net /GPIO6: track 0.00 -> 57.5 mm, vias 0 -> 1
- net /GPIO21(SPI1_SCK): track 0.00 -> 56.8 mm, vias 0 -> 1
- net EIO_2: track 0.00 -> 56.6 mm
- net /GPIO20(SPI1_MOSI): track 0.00 -> 48.7 mm, vias 0 -> 1
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Other:
- board text added: "Dumper Py"
- board text added: "https://github.com/km1ab/fc-dumper-py"

Commit message: add QR code to botom-PCB
Parts:
- added G***: LOGO, SamacSys_Parts:QR_code_8_5, F.Cu at (147.6, 58.1)

Commit message: add version silk
Other:
- board text added: "202212"
- board text added: "Rev1.0"
Changed lines of the file:
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@@
+    (effects (font (size 1 1) (thickness 0.15)))
+  )
+  (gr_text "202212" (at 146.99 63.17) (layer "F.SilkS")
     (effects (font (size 1 1) (thickness 0.15)))
   )
@@
     (effects (font (size 2 2) (thickness 0.3)))
   )
+  (gr_text "Rev1.0" (at 127.305 54.915) (layer "F.SilkS")
+    (effects (font (size 1 1) (thickness 0.15)))
+  )
   (gr_text "USB" (at 177.724 71.552) (layer "Dwgs.User")
