File: hat-prot-02/hat-prot-02.kicad_sch (KiCad schematic)
At the start: 18 parts, among them J1 Conn_01x10_Male, J2 Conn_01x12_Male, J3 Conn_01x05_Male, J4 CR22A-60D-2.54DS_70_, J5 SolderJumper_2_Open, J6 SolderJumper_2_Open, J7 SolderJumper_2_Open, Q1 2SC1815, Q2 2SC1815, SW1 SW_SPDT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

Commit message: modify design delete copy add QR code
Parts:
- removed J1: Conn_01x10_Male, Connector_PinSocket_2.54mm:PinSocket_1x10_P2.54mm_Vertical, symbol Connector:Conn_01x10_Male
- removed J2: Conn_01x12_Male, Connector_PinSocket_2.54mm:PinSocket_1x12_P2.54mm_Vertical, symbol Connector:Conn_01x12_Male
- removed J3: Conn_01x05_Male, Connector_PinHeader_2.54mm:PinHeader_1x05_P2.54mm_Vertical, symbol Connector:Conn_01x05_Male
- added J1: Conn_01x10_Female, Connector_PinSocket_2.54mm:PinSocket_1x10_P2.54mm_Vertical, symbol Connector:Conn_01x10_Female
- added J2: Conn_01x12_Female, Connector_PinSocket_2.54mm:PinSocket_1x12_P2.54mm_Vertical, symbol Connector:Conn_01x12_Female
- added J3: Conn_02x04_Odd_Even, Connector_PinHeader_2.54mm:PinHeader_2x04_P2.54mm_Vertical, symbol Connector_Generic:Conn_02x04_Odd_Even
- added J4: Conn_01x04_Female, Connector_PinSocket_2.54mm:PinSocket_1x04_P2.54mm_Vertical, symbol Connector:Conn_01x04_Female
- renumbered J4 to J5, J5 to JP1, J6 to JP2, J7 to JP3
Connections:
- net ADR13: now also J5.B26
- net CLK: now also J2.6 (Pin_6)
- net CLR: now also J2.7 (Pin_7)
- net CS: now also J2.3 (Pin_3)
- net DA0: now also J1.1 (Pin_1)
- net DA1: now also J1.2 (Pin_2)
- net DA2: now also J1.3 (Pin_3)
- net DA3: now also J1.4 (Pin_4)
- net DA4: now also J1.5 (Pin_5)
- net DA5: now also J1.6 (Pin_6)
- net DA6: now also J1.7 (Pin_7)
- net DA7: now also J1.8 (Pin_8)
- net EIO_0: now also J2.11 (Pin_11), J3.3 (Pin_3)
- net EIO_1: now also J3.5 (Pin_5), J4.1 (Pin_1)
- net EIO_2: now also J3.7 (Pin_7), J4.2 (Pin_2)
- net GND: now also J2.12 (Pin_12), J3.8 (Pin_8)
- net OE: now also J2.2 (Pin_2)
- net PWM0: now also J1.9 (Pin_9)
- net PWM1: now also J1.10 (Pin_10)
- net PWR: now also J5.A30, J5.B1
- net PWR3: now also J2.10 (Pin_10), J3.1 (Pin_1)
- net VIN: now also J2.1 (Pin_1); no longer J5.A30, J5.B1
- net WE: now also J2.4 (Pin_4); no longer J5.B17
- net ADR15 renamed PPU/A13
- net RST renamed PPURD
- net PPURD: now also J2.5 (Pin_5); no longer J5.B26
- new net EIO_3: J3.2 (Pin_2), J4.3 (Pin_3)
- new net EIO_4: J3.4 (Pin_4), J4.4 (Pin_4)
- new net EXT: J2.9 (Pin_9), J3.6 (Pin_6)
- new net PPUWR: J2.8 (Pin_8), J5.B17
